File: schematics/selfbalancingrobot.kicad_pcb (KiCad board)
At the start: 2 copper layers, 73.7 x 121.9 mm, 62 parts, among them IC1 SN754410, J1 POWER, J2 MOT-LEFT, J3 MOT-RIGHT, J4 ICSP, J5 ESP-RS232, J6 MOT-POWER, J7 DEBUG-TX, Q1 BC547, Q2 BC547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

Commit message: - Refinado PCB
Parts:
- C1, C4, C5, C8: footprint pth-passive:C-ALUM-8mm -> selfbalancingrobot:C-ALUM-8mm
- C2, C6, C7: footprint pth-passive:C-FILM-2.5mm -> selfbalancingrobot:C-FILM-2.5mm
- C3: footprint pth-passive:C-ALUM-5mm -> selfbalancingrobot:C-ALUM-5mm
- D1, D2, D3, D4: footprint pth-semi:DO-35 -> selfbalancingrobot:DO-35
- DS1, DS2, DS3, DS4: footprint pth-semi:LED-3mm -> selfbalancingrobot:LED-3mm
- IC1: footprint dip-sip:DIP-16 -> selfbalancingrobot:DIP-16
- J1, J6: footprint conn-100mil:CONN-100MIL-M-1x2-SHROUD -> selfbalancingrobot:CONN-100MIL-M-1x2-SHROUD
- J2, J3, J4: footprint conn-100mil:CONN-100MIL-M-1x6-SHROUD -> selfbalancingrobot:CONN-100MIL-M-1x6-SHROUD
- J5: footprint conn-100mil:CONN-100MIL-F-1x5 -> selfbalancingrobot:CONN-100MIL-F-1x5
- J7: footprint conn-100mil:CONN-100MIL-M-1x1 -> selfbalancingrobot:CONN-100MIL-M-1x1
- Q1, Q2: footprint pth-semi:TO-92 -> selfbalancingrobot:TO-92
- R1, R10, R11, R12, R13, R14, R15, R16, R17, R18, R19, R2, R20, R21, R22, R3, R4, R5, R6, R7, R8, R9: footprint pth-passive:R-250mW -> selfbalancingrobot:R-250mW
- SW1, SW2, SW3: footprint Buttons_Switches_THT:SW_PUSH_6mm_h5mm -> selfbalancingrobot:SW_PUSH_6mm_h5mm
- U1, U3: footprint pth-semi:TO-220 -> selfbalancingrobot:TO-220
- U2: footprint dip-sip:DIP-28 -> selfbalancingrobot:DIP-28
- U4: footprint ESP8266:ESP-12 -> selfbalancingrobot:ESP-12
- U5: footprint proj:MPU9265_breakout -> selfbalancingrobot:MPU9265_breakout
- renumbered REF** to 3,3V, REF** to ?
Routing:
- net GND: track 726.3 -> 739.1 mm
- net +3.3: track 379.4 -> 378.9 mm
Other:
- board text added: "12V"
- board text added: "7V"
- board text added: "GND"
- board text added: "SERIAL DEBUG"
- board text added: "SelfBalancing Robot v1.0 A. & G. Corp."
