File: schematics/selfbalancingrobot.kicad_pcb (KiCad board)
At the start: 2 copper layers, 73.7 x 121.9 mm, 62 parts, among them IC1 SN754410, J1 POWER, J2 MOT-LEFT, J3 MOT-RIGHT, J4 ICSP, J5 ESP-RS232, J6 MOT-POWER, J7 DEBUG-TX, Q1 BC547, Q2 BC547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

Commit message: - Mejorada señalización por leds en PIC y ESP8266
- ESP8266: Un error de la conexión a la Wifi permite continuar el programa
Parts:
- moved R9 0.18 mm to (156.0, 76.8)
Routing:
- net Net-(R21-Pad2): track 12.7 -> 14.4 mm
- net Net-(R22-Pad2): track 11.9 -> 13.3 mm
- net /MOT_LEFT_DIR0: track 30.2 -> 31.0 mm
Other:
- net class Default: clearance 0.381 -> 0.508
- net class Power: clearance 0.381 -> 0.508
- rule trace_clearance: 0.381 -> 0.508
- board text added: "SelfBalancing Robot v1.0 A. & G. Corp. 14/10/2017"
- board text removed: "SelfBalancing Robot v1.0 A. & G. Corp."
